Commit message: - FIx wrong val in urdf,  refine kinematics and controllers configuration for dual arm RM65

File: rm_description/urdf/dual_rm65.urdf (robot description, URDF)
Before this commit: robot dual_rm65, 15 links, 14 joints
Joints:
- joint left_joint1: origin xyz=0 0 0 rpy=0 0 0 -> xyz=0 0 0.2405 rpy=0 0 0
- joint right_joint1: origin xyz=0 0 0 rpy=0 0 0 -> xyz=0 0 0.2405 rpy=0 0 0
