Commit message: - Add robotiq_2f85 gripper model

File: rm_description/urdf/rm65_arm_macro.xacro (robot description, xacro)
@@ -27,5 +27,5 @@
     <!-- joint1 连接到这个独立的 base_link -->
     <joint name="${prefix}joint1" type="revolute">
-      <origin xyz="0 0 0" rpy="0 0 0"/>
+      <origin xyz="0 0 0.2405" rpy="0 0 0"/>
       <parent link="${prefix}base_link"/>
       <child link="${prefix}Link1"/>

File: rm_moveit2_config/dual_arm_rm_65_config/config/dual_rm65.urdf.xacro (robot description, xacro)
@@ -7,3 +7,16 @@
     <xacro:include filename="dual_rm65.ros2_control.xacro" />
     <xacro:dual_rm65_ros2_control name="FakeSystem" initial_positions_file="$(arg initial_positions_file)"/>
+    <!-- Gripper macro definitions -->
+    <xacro:include filename="$(find robotiq_2f85_description)/robots/robotiq_2f85_gripper.xacro" />
+    <!-- robotiq_2f85 -->
+    <xacro:robotiq_2f85_gripper
+            prefix="left_gripper_"
+            parent="left_Link6"
+            xyz="0 0 0"
+            rpy="0 0 0" />
+    <xacro:robotiq_2f85_gripper
+        prefix="right_gripper_"
+        parent="right_Link6"
+        xyz="0 0 0"
+        rpy="0 0 -${pi/6}" />
 </robot>
