Commit message: - Remove unused urdf, configure urdf mounting and base offset via xacro marco

File: rm_moveit2_config/dual_arm_rm_65_config/config/dual_rm65.srdf.xacro (robot description, xacro)
@@ -15,4 +15,6 @@
     <xacro:arg name="gripper" default="robotiq_2f85" />
     <xacro:property name="gripper_type" value="$(arg gripper)" />
+    <xacro:property name="left_tip_link" value="${'left_gripper_tcp' if gripper_type == 'robotiq_2f85' else 'left_Link6'}" />
+    <xacro:property name="right_tip_link" value="${'right_gripper_tcp' if gripper_type == 'robotiq_2f85' else 'right_Link6'}" />
     <!-- ══════════════════════════════════════════════════════════════
          GRIPPER COLLISION MACRO
@@ -56,8 +58,8 @@
          ══════════════════════════════════════════════════════════════ -->
     <group name="left_arm">
-        <chain base_link="left_base_link" tip_link="left_Link6"/>
+        <chain base_link="left_base_link" tip_link="${left_tip_link}"/>
     </group>
     <group name="right_arm">
-        <chain base_link="right_base_link" tip_link="right_Link6"/>
+        <chain base_link="right_base_link" tip_link="${right_tip_link}"/>
     </group>
     <group name="dual_arm">

File: rm_moveit2_config/dual_arm_rm_65_config/config/dual_rm65.urdf.xacro (robot description, xacro)
@@ -3,5 +3,5 @@
     <xacro:arg name="initial_positions_file" default="initial_positions.yaml" />
     <!-- Import dual_rm65 urdf file -->
-    <xacro:include filename="$(find rm_description)/urdf/dual_rm65.urdf" />
+    <xacro:include filename="$(find rm_description)/urdf/dual_rm65.urdf.xacro" />
     <!-- Import control_xacro -->
     <xacro:include filename="dual_rm65.ros2_control.xacro" />
@@ -14,9 +14,13 @@
             parent="left_Link6"
             xyz="0 0 0"
-            rpy="0 0 0" />
+            rpy="0 0 -${pi/4}"
+            tcp_xyz="0 0 0.17"
+            tcp_rpy="0 0 0" />
     <xacro:robotiq_2f85_gripper
         prefix="right_gripper_"
         parent="right_Link6"
         xyz="0 0 0"
-        rpy="0 0 -${pi/6}" />
+        rpy="0 0 ${pi*5/12}"
+        tcp_xyz="0 0 0.17"
+        tcp_rpy="0 0 0" />
 </robot>
